File: Altimeter.kicad_sch (KiCad schematic)
At the start: 27 parts, among them IC1 XC9801B503KR-G, IC2 ATTINY804-SSF, IC3 MC3479, IC4 MCP73855-I_MF, IC5 XC9265B181MR-G, J1 USB3075-30-A, J2 Battery, J3 Conn_01x03_Female, U1 ICP-10111

Commit message: no done
Parts:
- J3: footprint Connector_PinHeader_2.00mm:PinHeader_1x03_P2.00mm_Vertical -> Connector_PinHeader_2.54mm:PinHeader_1x03_P2.54mm_Vertical
Changed lines of the file:
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@@
   (symbol (lib_id "power:Earth") (at 95.25 52.07 270) (unit 1)
     (in_bom yes) (on_board yes) (fields_autoplaced)
-    (property "Reference" "#PWR?" (id 0) (at 88.9 52.07 0)
+    (property "Reference" "#PWR0127" (id 0) (at 88.9 52.07 0)
       (effects (font (size 1.27 1.27)) hide)
     )
@@
       (effects (font (size 1.27 1.27)) (justify left))
     )
-    (property "Footprint" "Connector_PinHeader_2.00mm:PinHeader_1x03_P2.00mm_Vertical" (id 2) (at 142.24 138.43 0)
+    (property "Footprint" "Connector_PinHeader_2.54mm:PinHeader_1x03_P2.54mm_Vertical" (id 2) (at 142.24 138.43 0)
       (effects (font (size 1.27 1.27)) hide)
     )
@@
     )
     (path "/84969346-7f67-4be5-9178-143d78a1823f"
-      (reference "#PWR?") (unit 1) (value "Earth") (footprint "")
+      (reference "#PWR0127") (unit 1) (value "Earth") (footprint "")
     )
     (path "/37cf9889-35f0-4322-8722-2a0e92e7a23f"
@@
     )
     (path "/b098508d-025c-4022-80c4-639f79b6b495"
-      (reference "J3") (unit 1) (value "Conn_01x03_Female") (footprint "Connector_PinHeader_2.00mm:PinHeader_1x03_P2.00mm_Vertical")
+      (reference "J3") (unit 1) (value "Conn_01x03_Female") (footprint "Connector_PinHeader_2.54mm:PinHeader_1x03_P2.54mm_Vertical")
     )
     (path "/1eb279b8-cfeb-41b6-8510-73a87163ce55"
