File: Altimeter.kicad_sch (KiCad schematic)
At the start: 28 parts, among them IC1 XC9801B503KR-G, IC2 ATTINY804-SSF, IC3 MC3479, IC4 MCP73855-I_MF, IC5 XC9265B181MR-G, J1 USB3075-30-A, J2 Battery, J3 Conn_01x03_Female, U1 ICP-10111

Commit message: changes
Parts:
- J2: footprint Connector_PinHeader_2.54mm:PinHeader_1x03_P2.54mm_Vertical -> Connector_PinHeader_2.54mm:PinHeader_1x04_P2.54mm_Vertical; symbol Connector:Conn_01x03_Female -> Connector:Conn_01x04_Female
Connections:
- net BAT: now also J2.3 (Pin_3)
- net Earth: now also J2.4 (Pin_4); no longer J2.3 (Pin_3)
Changed lines of the file:
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@@
   (junction (at 168.91 54.61) (diameter 0) (color 0 0 0 0)
   )
+  (junction (at 137.16 151.13) (diameter 0) (color 0 0 0 0)
+  )
   (wire (pts (xy 204.47 54.61) (xy 204.47 57.15))
     (stroke (width 0) (type default) (color 0 0 0 0))
@@
   )
   (wire (pts (xy 166.37 54.61) (xy 168.91 54.61))
+    (stroke (width 0) (type default) (color 0 0 0 0))
+  )
+  (wire (pts (xy 137.16 151.13) (xy 137.16 153.67))
     (stroke (width 0) (type default) (color 0 0 0 0))
   )
@@
     (pin "8")
   )
-  (symbol (lib_id "Connector:Conn_01x03_Female") (at 142.24 151.13 0) (unit 1)
+  (symbol (lib_id "Connector:Conn_01x04_Female") (at 142.24 151.13 0) (unit 1)
     (in_bom yes) (on_board yes) (fields_autoplaced)
     (property "Reference" "J2" (id 0) (at 143.51 151.1299 0)
@@
       (effects (font (size 1.27 1.27)) (justify left))
     )
-    (property "Footprint" "Connector_PinHeader_2.54mm:PinHeader_1x03_P2.54mm_Vertical" (id 2) (at 142.24 151.13 0)
+    (property "Footprint" "Connector_PinHeader_2.54mm:PinHeader_1x04_P2.54mm_Vertical" (id 2) (at 142.24 151.13 0)
       (effects (font (size 1.27 1.27)) hide)
     )
@@
     (pin "2")
     (pin "3")
+    (pin "4")
   )
   (symbol (lib_id "power:Earth") (at 138.43 44.45 90) (unit 1)
@@
     (pin "1")
   )
-  (symbol (lib_id "power:Earth") (at 137.16 153.67 270) (unit 1)
-    (in_bom yes) (on_board yes) (fields_autoplaced)
-    (property "Reference" "#PWR01" (id 0) (at 130.81 153.67 0)
-      (effects (font (size 1.27 1.27)) hide)
-    )
-    (property "Value" "Earth" (id 1) (at 133.35 153.67 0)
-      (effects (font (size 1.27 1.27)) hide)
-    )
-    (property "Footprint" "" (id 2) (at 137.16 153.67 0)
-      (effects (font (size 1.27 1.27)) hide)
-    )
-    (property "Datasheet" "~" (id 3) (at 137.16 153.67 0)
+  (symbol (lib_id "power:Earth") (at 137.16 156.21 270) (unit 1)
+    (in_bom yes) (on_board yes) (fields_autoplaced)
+    (property "Reference" "#PWR01" (id 0) (at 130.81 156.21 0)
+      (effects (font (size 1.27 1.27)) hide)
+    )
+    (property "Value" "Earth" (id 1) (at 133.35 156.21 0)
+      (effects (font (size 1.27 1.27)) hide)
+    )
+    (property "Footprint" "" (id 2) (at 137.16 156.21 0)
+      (effects (font (size 1.27 1.27)) hide)
+    )
+    (property "Datasheet" "~" (id 3) (at 137.16 156.21 0)
       (effects (font (size 1.27 1.27)) hide)
     )
@@
     )
     (path "/0a55cbbb-2ce0-40e3-849c-00aae905b08b"
-      (reference "J2") (unit 1) (value "Battery") (footprint "Connector_PinHeader_2.54mm:PinHeader_1x03_P2.54mm_Vertical")
+      (reference "J2") (unit 1) (value "Battery") (footprint "Connector_PinHeader_2.54mm:PinHeader_1x04_P2.54mm_Vertical")
     )
     (path "/b098508d-025c-4022-80c4-639f79b6b495"

Commit message: changes
Parts:
- removed C3: .5uF, Capacitor_SMD:C_0805_2012Metric_Pad1.18x1.45mm_HandSolder, symbol Device:C_Small
- removed IC1: XC9801B503KR-G, SamacSys_Parts:SOP65P490X122-8N, symbol SamacSys_Parts:XC9801B503KR-G
- added IC1: DIO6605BFN8, SamacSys_Parts:SON50P300X200X80-9N-D, symbol SamacSys_Parts:DIO6605BFN8
- added L2: 4.7uF, Inductor_SMD:L_0805_2012Metric_Pad1.05x1.20mm_HandSolder, symbol Device:L
- C1, C2: value 5uF -> 10uF
Connections:
- net BAT: now also IC1.5 (VIN), L2.1
- net BUZZER: now also IC1.1 (EN)
- net Earth: now also IC1.2 (AGND), IC1.3 (PGND), IC1.9 (GND)
- net at C2.1, LS1.1 (+): now also IC1.7 (VOUT)
- new net: IC1.4 (SW), L2.2
Other:
- moved on the sheet: C1, C2, LS1
