File: Altimeter.kicad_pcb (KiCad board)
At the start: 2 copper layers, 12.8 x 49.7 mm, 27 parts, among them IC1 XC9801B503KR-G, IC2 ATTINY804-SSF, IC3 MC3479, IC4 MCP73855-I_MF, IC5 XC9265B181MR-G, J1 USB3075-30-A, J2 Battery, J3 Conn_01x03_Female, U1 ICP-10111

Commit message: no done
Parts:
- J3: footprint Connector_PinHeader_2.00mm:PinHeader_1x03_P2.00mm_Vertical -> Connector_PinHeader_2.54mm:PinHeader_1x03_P2.54mm_Vertical
- moved J3 0.49 mm to (36.3, 72.0)

Commit message: final?
Routing:
- net /5V: track 40.5 -> 45.5 mm, vias 2 -> 4
- net Earth: vias 3 -> 6
Changed lines of the file:
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@@
     (property "Sheetname" "")
     (attr through_hole)
-    (fp_text reference "J1" (at 0 -0.6) (layer "F.SilkS")
+    (fp_text reference "J1" (at 0 2.233) (layer "F.SilkS")
       (effects (font (size 1.27 1.27) (thickness 0.254)))
     )
@@
     (property "Sheetname" "")
     (attr through_hole)
-    (fp_text reference "J2" (at 0 -2.06 90) (layer "F.SilkS")
+    (fp_text reference "J2" (at 1.696 0.005 90) (layer "F.SilkS")
       (effects (font (size 1 1) (thickness 0.15)))
     )
@@
     (property "Sheetname" "")
     (attr smd)
-    (fp_text reference "C4" (at 0 1.68 90) (layer "B.SilkS")
+    (fp_text reference "C4" (at -0.161 -1.454 90) (layer "B.SilkS")
       (effects (font (size 1 1) (thickness 0.15)) (justify mirror))
     )
@@
     (property "Sheetname" "")
     (attr smd)
-    (fp_text reference "C5" (at 0 1.68 90) (layer "B.SilkS")
+    (fp_text reference "C5" (at -0.082 -1.647 90) (layer "B.SilkS")
       (effects (font (size 1 1) (thickness 0.15)) (justify mirror))
     )
@@
     (property "Sheetname" "")
     (attr smd)
-    (fp_text reference "IC3" (at 0 0) (layer "B.SilkS")
+    (fp_text reference "IC3" (at 0.798 -2.412) (layer "B.SilkS")
       (effects (font (size 1.27 1.27) (thickness 0.254)) (justify mirror))
     )
@@
     (property "Sheetname" "")
     (attr smd)
-    (fp_text reference "IC1" (at 0 0) (layer "B.SilkS")
+    (fp_text reference "IC1" (at 0 -0.214) (layer "B.SilkS")
       (effects (font (size 1.27 1.27) (thickness 0.254)) (justify mirror))
     )
@@
     (property "Sheetname" "")
     (attr smd)
-    (fp_text reference "C10" (at 0 1.85 90) (layer "B.SilkS")
+    (fp_text reference "C10" (at 3.978 1.061 90) (layer "B.SilkS")
       (effects (font (size 1 1) (thickness 0.15)) (justify mirror))
     )
@@
     (property "Sheetname" "")
     (attr smd)
-    (fp_text reference "C2" (at 0 1.68 90) (layer "B.SilkS")
+    (fp_text reference "C2" (at -1.062 4.234 90) (layer "B.SilkS")
       (effects (font (size 1 1) (thickness 0.15)) (justify mirror))
     )
@@
     (property "Sheetname" "")
     (attr smd)
-    (fp_text reference "R1" (at 2.564 -3.297) (layer "B.SilkS")
+    (fp_text reference "R1" (at -3.084 1.029) (layer "B.SilkS")
       (effects (font (size 1 1) (thickness 0.15)) (justify mirror))
     )
@@
     (property "Sheetname" "")
     (attr smd)
-    (fp_text reference "C7" (at 0 1.85 90) (layer "B.SilkS")
+    (fp_text reference "C7" (at 2.268 1.637 90) (layer "B.SilkS")
       (effects (font (size 1 1) (thickness 0.15)) (justify mirror))
     )
@@
     (property "Sheetname" "")
     (attr smd)
-    (fp_text reference "L1" (at 0 1.9 90) (layer "B.SilkS")
+    (fp_text reference "L1" (at -3.478 2.679 90) (layer "B.SilkS")
       (effects (font (size 1 1) (thickness 0.15)) (justify mirror))
     )
@@
     (property "Sheetname" "")
     (attr smd)
-    (fp_text reference "U1" (at 0.45 0) (layer "B.SilkS")
+    (fp_text reference "U1" (at -1.552 2.534) (layer "B.SilkS")
       (effects (font (size 1.27 1.27) (thickness 0.254)) (justify mirror))
     )
@@
     (property "Sheetname" "")
     (attr smd)
-    (fp_text reference "R2" (at 0 1.65) (layer "B.SilkS")
+    (fp_text reference "R2" (at 0.079 -1.671) (layer "B.SilkS")
       (effects (font (size 1 1) (thickness 0.15)) (justify mirror))
     )
@@
     (property "Sheetname" "")
     (attr smd)
-    (fp_text reference "C8" (at 0.127 1.651 90) (layer "B.SilkS")
+    (fp_text reference "C8" (at 0 -1.814 90) (layer "B.SilkS")
       (effects (font (size 1 1) (thickness 0.15)) (justify mirror))
     )
@@
     (property "Sheetname" "")
     (attr smd)
-    (fp_text reference "R3" (at 0 1.65) (layer "B.SilkS")
+    (fp_text reference "R3" (at 0.878 1.578) (layer "B.SilkS")
       (effects (font (size 1 1) (thickness 0.15)) (justify mirror))
     )
@@
     (property "Sheetname" "")
     (attr smd)
-    (fp_text reference "IC5" (at 0 0) (layer "B.SilkS")
+    (fp_text reference "IC5" (at 0.181 -2.368) (layer "B.SilkS")
       (effects (font (size 1.27 1.27) (thickness 0.254)) (justify mirror))
     )
@@
     (property "Sheetname" "")
     (attr smd)
-    (fp_text reference "R4" (at 0 1.65) (layer "B.SilkS")
+    (fp_text reference "R4" (at 0 1.422) (layer "B.SilkS")
       (effects (font (size 1 1) (thickness 0.15)) (justify mirror))
     )
@@
   )
   (gr_rect (start 32.831 46.228) (end 44.831 73.228) (layer "F.SilkS") (width 0.15) (fill none))
+  (gr_line (start 40.1 42.8) (end 40.1 43.6) (layer "F.SilkS") (width 0.15))
+  (gr_line (start 37.6 43.3) (end 38.4 43.3) (layer "F.SilkS") (width 0.15))
+  (gr_line (start 39.7 43.2) (end 40.5 43.2) (layer "F.SilkS") (width 0.15))
   (gr_rect (start 32.512 73.533) (end 45.339 23.876) (layer "Edge.Cuts") (width 0.1) (fill none))
+  (via (at 38.2 43.1) (size 0.46) (drill 0.2) (layers "F.Cu" "B.Cu") (free) (net 1))
   (via (at 39.497 55.753) (size 0.46) (drill 0.2) (layers "F.Cu" "B.Cu") (free) (net 1))
+  (via (at 38.1 41.7) (size 0.46) (drill 0.2) (layers "F.Cu" "B.Cu") (free) (net 1))
+  (via (at 41.8 34.7) (size 0.46) (drill 0.2) (layers "F.Cu" "B.Cu") (free) (net 1))
   (via (at 41.656 58.039) (size 0.46) (drill 0.2) (layers "F.Cu" "B.Cu") (free) (net 1))
   (via (at 43.561 38.989) (size 0.46) (drill 0.2) (layers "F.Cu" "B.Cu") (free) (net 1))
@@
   (segment (start 45.085 55.118) (end 45.085 55.753) (width 0.2) (layer "B.Cu") (net 6))
   (segment (start 37.465 31.877) (end 37.465 30.988) (width 0.25) (layer "F.Cu") (net 7))
-  (segment (start 33.909 24.765) (end 33.909 30.607) (width 0.2) (layer "F.Cu") (net 7))
+  (segment (start 34.5 26.7) (end 33.918 26.7) (width 0.2) (layer "F.Cu") (net 7))
+  (segment (start 33.909 24.765) (end 33.909 26.691) (width 0.2) (layer "F.Cu") (net 7))
   (segment (start 34.29 30.988) (end 37.465 30.988) (width 0.2) (layer "F.Cu") (net 7))
   (segment (start 33.646 44.441) (end 33.51 44.577) (width 0.2) (layer "F.Cu") (net 7))
   (segment (start 33.646 35.696) (end 33.646 44.441) (width 0.2) (layer "F.Cu") (net 7))
+  (segment (start 33.909 26.691) (end 33.909 30.607) (width 0.2) (layer "F.Cu") (net 7))
   (segment (start 33.909 30.607) (end 34.29 30.988) (width 0.2) (layer "F.Cu") (net 7))
+  (segment (start 37.943 25.417) (end 37.943 26.443) (width 0.2) (layer "F.Cu") (net 7))
   (segment (start 41.402 30.988) (end 41.783 31.369) (width 0.25) (layer "F.Cu") (net 7))
+  (segment (start 37.943 26.443) (end 38.1 26.6) (width 0.2) (layer "F.Cu") (net 7))
   (segment (start 37.943 24.917) (end 37.537 24.511) (width 0.2) (layer "F.Cu") (net 7))
   (segment (start 37.465 30.988) (end 41.402 30.988) (width 0.25) (layer "F.Cu") (net 7))
-  (segment (start 37.943 25.417) (end 37.943 24.917) (width 0.2) (layer "F.Cu") (net 7))
+  (segment (start 33.918 26.7) (end 33.909 26.691) (width 0.2) (layer "F.Cu") (net 7))
   (segment (start 37.537 24.511) (end 34.163 24.511) (width 0.2) (layer "F.Cu") (net 7))
   (segment (start 41.783 31.369) (end 41.783 33.528) (width 0.25) (layer "F.Cu") (net 7))
   (segment (start 33.646 35.696) (end 37.465 31.877) (width 0.2) (layer "F.Cu") (net 7))
   (segment (start 34.163 24.511) (end 33.909 24.765) (width 0.2) (layer "F.Cu") (net 7))
+  (via (at 34.5 26.7) (size 0.46) (drill 0.2) (layers "F.Cu" "B.Cu") (net 7))
+  (via (at 38.1 26.6) (size 0.46) (drill 0.2) (layers "F.Cu" "B.Cu") (net 7))
   (via (at 37.465 31.877) (size 0.46) (drill 0.2) (layers "F.Cu" "B.Cu") (net 7))
   (via (at 41.783 33.528) (size 0.46) (drill 0.2) (layers "F.Cu" "B.Cu") (net 7))
+  (segment (start 38 26.7) (end 34.5 26.7) (width 0.2) (layer "B.Cu") (net 7))
   (segment (start 37.489 31.901) (end 37.465 31.877) (width 0.25) (layer "B.Cu") (net 7))
+  (segment (start 38.1 26.6) (end 38 26.7) (width 0.2) (layer "B.Cu") (net 7))
   (segment (start 42.2695 33.528) (end 43.053 32.7445) (width 0.25) (layer "B.Cu") (net 7))
   (segment (start 40.489 33.504) (end 40.489 33.282) (width 0.25) (layer "B.Cu") (net 7))

Commit message: maybe actual final
Parts:
- added C11: .1uF, Capacitor_SMD:C_0805_2012Metric_Pad1.18x1.45mm_HandSolder, B.Cu at (44.0, 60.1)
- C1: value 1uF -> 5uF
- J2: footprint Connector_PinHeader_2.00mm:PinHeader_1x02_P2.00mm_Vertical -> Connector_PinHeader_2.54mm:PinHeader_1x03_P2.54mm_Vertical
- R5: value 100 -> 250
- moved D1 16.9 mm to (33.6, 27.7), turned to 90 degrees
- moved R5 16.4 mm to (33.6, 31.5), turned to -90 degrees
- moved J1 1.35 mm to (39.7, 26.8), turned to 180 degrees
- moved C7 0.71 mm to (34.4, 48.1)
- moved L1 0.24 mm to (41.1, 48.8)
- moved C10 0.22 mm to (43.6, 48.8)
Connections:
- J2 pad 2: Earth -> /BAT
Routing:
- net /5V: track 45.5 -> 19.3 mm, vias 4 -> 2
- net Net-(IC4-Pad1): track 18.5 -> 7.53 mm
- net Net-(D1-Pad1): track 10.5 -> 1.77 mm
- net Earth: track 3.41 -> 11.5 mm, vias 6 -> 14
- net /1.8V: track 39.9 -> 42.5 mm
Other:
- board size 12.8 x 49.7 mm -> 12.8 x 48.3 mm
