File: Altimeter.kicad_pcb (KiCad board)
At the start: 2 copper layers, 12.8 x 48.3 mm, 28 parts, among them IC1 XC9801B503KR-G, IC2 ATTINY804-SSF, IC3 MC3479, IC4 MCP73855-I_MF, IC5 XC9265B181MR-G, J1 USB3075-30-A, J2 Battery, J3 Conn_01x03_Female, U1 ICP-10111

Commit message: changes
Parts:
- J2: footprint Connector_PinHeader_2.54mm:PinHeader_1x03_P2.54mm_Vertical -> Connector_PinHeader_2.54mm:PinHeader_1x04_P2.54mm_Vertical
- moved J2 1.80 mm to (41.8, 44.7)
- moved C1 0.89 mm to (44.1, 42.7), turned to 90 degrees
Connections:
- J2 pad 3: Earth -> /BAT
Routing:
- net Earth: track 11.5 -> 1.48 mm, vias 14 -> 23
- net /BAT: track 56.3 -> 55.1 mm, vias 3 -> 5

Commit message: changes
Parts:
- removed C3: .5uF, Capacitor_SMD:C_0805_2012Metric_Pad1.18x1.45mm_HandSolder
- added L2: 4.7uF, Inductor_SMD:L_0805_2012Metric_Pad1.05x1.20mm_HandSolder, B.Cu at (40.7, 42.5)
- C1, C2: value 5uF -> 10uF
- IC1: value XC9801B503KR-G -> DIO6605BFN8; footprint SamacSys_Parts:SOP65P490X122-8N -> SamacSys_Parts:SON50P300X200X80-9N-D
- moved C2 8.51 mm to (35.2, 40.8)
- moved C1 2.42 mm to (42.9, 40.6), turned to 180 degrees
- moved IC1 0.64 mm to (38.6, 40.4)
Connections:
- IC1 pad 1: Net-(C2-Pad1) -> /BUZZER
- IC1 pad 2: /BUZZER -> Earth
- IC1 pad 3: /BAT -> Earth
- IC1 pad 4: Earth -> Net-(IC1-Pad4)
- IC1 pad 5: Earth -> /BAT
- IC1 pad 6: Net-(C3-Pad2) -> unconnected-(IC1-Pad6)
- IC1 pad 7: Net-(C3-Pad1) -> Net-(C2-Pad1)
- IC1 pad 8: Net-(C2-Pad1) -> unconnected-(IC1-Pad8)
Routing:
- net /BAT: track 55.1 -> 59.5 mm
- net Net-(C3-Pad2): track 2.46 -> 0.00 mm
- net Net-(C2-Pad1): track 11.8 -> 9.53 mm
- net Net-(C3-Pad1): track 2.02 -> 0.00 mm
- net Net-(IC1-Pad4): track 0.00 -> 1.62 mm
- net /BUZZER: track 30.4 -> 29.3 mm
- net Earth: track 1.48 -> 0.95 mm, vias 23 -> 26

Commit message: changes
Parts:
- moved C9 1.78 mm to (33.6, 35.3)
- moved C5 0.84 mm to (42.2, 33.6)
- moved L2 0.58 mm to (41.3, 42.6)
- moved C2 0.30 mm to (35.5, 40.8)
- moved C1 0.18 mm to (42.7, 40.7)
- moved C11 0.08 mm to (43.9, 60.1)
Routing:
- net Earth: track 0.95 -> 1.19 mm, vias 26 -> 30
